Commit message: Urdf setup completly

File: amr_swarming_description/urdf/robot.urdf.xacro (robot description, xacro)
@@ -1,70 +1,5 @@
-<?xml version = "1.0"?>
-<robot name="four_wheeled_differential_drive_robot"
-       xmlns:xacro="http://www.ros.org/wiki/xacro">
-    <!-- Properties -->
-    <xacro:property name = "robot_amr" value = "four_wheeled_differential_drive_robot"/>
-    <xacro:property name = "wheel_radius" value = "0.05"/>
-    <xacro:property name = "wheel_width" value = "0.02"/>
-    <xacro:property name = "chassis_length" value = "0.4"/>
-    <xacro:property name = "chassis_width" value = "0.3"/>
-    <xacro:property name = "chassis_height" value = "0.1"/>
-    <!-- BASE LINK (CHASSIS)-->
-    <link name = "base_link">
-        <visual>
-            <geometry>
-                <box size = "${chassis_length} ${chassis_width} ${chassis_height}"/>
-            </geometry>
-            <origin xyz= "0 0 ${chassis_height/2}" rpy = "0 0 0"/>
-            <material name = "red">
-                <color rgba = "1 0.0 0.0 1.0"/>
-            </material>
-        </visual>
-        <collision>
-            <geometry>
-                <box size = "${chassis_length} ${chassis_width} ${chassis_height}"/>
-            </geometry>
-            <origin xyz= "0 0 ${chassis_height/2}" rpy = "0 0 0"/>
-        </collision>
-        <inertial>
-            <origin xyz= "0 0 0" rpy = "0 0 0"/>
-            <mass value = "5.0"/>
-            <inertia ixx = "0.1" ixy = "0.0" ixz = "0.0" iyy = "0.1" iyz= "0.0" izz = "0.1"/>
-        </inertial>
-    </link>
-    <!-- WHEELS MACRO -->
-    <xacro:macro name = "wheel" params = "prefix x y">
-        <link name = "${prefix}_wheel">
-            <visual>
-                <geometry>
-                <cylinder radius = "${wheel_radius}" length = "${wheel_width}"/>
-                </geometry>
-                <origin xyz= "0 0 0" rpy = "1.5708 0 0"/>
-                <material name = "black">
-                    <color rgba = "0.0 0.0 0.0 1.0"/>
-                </material>
-            </visual>
-            <collision>
-                <geometry>
-                    <cylinder radius = "${wheel_radius}" length = "${wheel_width}"/>
-                </geometry>
-                <origin xyz = "0 0 0" rpy = "1.5708 0 0"/>
-            </collision>
-            <inertial>
-                <origin xyz = "0 0 0" rpy = "0 0 0"/>
-                <mass value = "0.3"/>
-                <inertia ixx = "0.001" ixy = "0.0" ixz = "0.0" iyy = "0.001" iyz= "0.0" izz = "0.001"/>
-            </inertial>
-        </link>
-        <joint name = "${prefix}_wheel_joint" type = "continuous">
-            <parent link = "base_link"/>
-            <child link = "${prefix}_wheel"/>
-            <origin xyz = "${x} ${y} ${wheel_radius}" rpy = "0 0 0"/>
-            <axis xyz  = "0 0 1"/>
-        </joint>
-    </xacro:macro>
-    <!-- ======== 4 WHEELS ========= -->
-    <xacro:wheel prefix = "front_left" x = "0.15" y = "0.15"/>
-    <xacro:wheel prefix = "front_right" x = "0.15" y = "-0.15"/>
-    <xacro:wheel prefix = "rear_left" x = "-0.15" y = "0.15"/>
-    <xacro:wheel prefix = "rear_right" x = "-0.15" y = "-0.15"/>
+<?xml version="1.0"?>
+<robot name="four_wheeled_differential_drive_robot" xmlns:xacro="http://www.ros.org/wiki/xacro">
+    <xacro:include filename="common_properties.xacro"/>
+    <xacro:include filename="urdf_robot.xacro"/>
 </robot>
